File: Schematic/WeatherStation.kicad_pcb (KiCad board)
At the start: 2 copper layers, 271.8 x 185.4 mm, 74 parts, among them J1 SolarPanels, J10 ESP Connector, J11 Conn_01x02, J2 TowerPlug, J3 ICSP Header, J4 Conn_01x05, J5 BME Connector, J6 Lux Connector, J7 BME Connector, J8 Conn_01x05, J9 ESP Connector, Q1 FQP30N06L, Q2 FQP27P06, Q3 FQP27P06, Q4 FQP30N06L, Q5 FQP27P06, Q6 FQP30N06L, Q7 FQP27P06, SW1 SW_RESET, U1 MCP1826-ADJ, U2 TC4056A_BASED_CHARGER, U3 ATmega328P-PU, U4 BME280Breakout, U5 23LC1024, U6 NodeMCU_1.0_(ESP-12E), U7 MCP23008, U8 RTCModule, Y1 16MHz

Commit message: C : : Updated Schemati
Parts:
- added C4: 10uF, Capacitors_THT:C_Disc_D5.0mm_W2.5mm_P5.00mm, F.Cu at (43.2, 43.2)
- added J12: Rain_Conn, Connectors_JST:JST_XH_B02B-XH-A_02x2.50mm_Straight, F.Cu at (30.5, 33.0)
- added L1: 10uF, Inductors_THT:L_Axial_L5.3mm_D2.2mm_P7.62mm_Horizontal_Vishay_IM-1, F.Cu at (58.4, 83.8)
- added R22: 10K, Resistors_THT:R_Axial_DIN0207_L6.3mm_D2.5mm_P7.62mm_Horizontal, F.Cu at (106.7, 154.9)
- added R23: 1k, Resistors_THT:R_Axial_DIN0207_L6.3mm_D2.5mm_P5.08mm_Vertical, F.Cu at (35.6, 38.1)
- added R24: 10K, Resistors_THT:R_Axial_DIN0207_L6.3mm_D2.5mm_P5.08mm_Vertical, F.Cu at (45.7, 43.2)
- added U5: 23LC1024, Housings_DIP:DIP-8_W7.62mm, F.Cu at (48.3, 119.4)
- C1: value 100nF -> 10uF; footprint WeatherLibrary:C_Disc_D5.0mm_W2.5mm_P7.54mm -> Capacitors_THT:C_Disc_D5.0mm_W2.5mm_P5.00mm
- C15: footprint Capacitors_THT:C_Disc_D5.0mm_W2.5mm_P2.50mm -> Capacitors_THT:C_Disc_D5.0mm_W2.5mm_P5.00mm
- J3: footprint Pin_Headers:Pin_Header_Straight_1x04_Pitch2.54mm -> Pin_Headers:Pin_Header_Straight_1x05_Pitch2.54mm
- J6: footprint Connectors_JST:JST_XH_B04B-XH-A_04x2.50mm_Straight -> Connectors_JST:JST_XH_B05B-XH-A_05x2.50mm_Straight
- J9: footprint Connectors_JST:JST_XH_B06B-XH-A_06x2.50mm_Straight -> Connectors_JST:JST_XH_B07B-XH-A_07x2.50mm_Straight
- R14, R15: footprint Resistors_THT:R_Axial_DIN0207_L6.3mm_D2.5mm_P5.08mm_Vertical -> Resistors_THT:R_Axial_DIN0207_L6.3mm_D2.5mm_P15.24mm_Horizontal
- R16: footprint WeatherLibrary:R_Axial_DIN0207_L6.3mm_D2.5mm_P12.7mm_Horizontal -> Resistors_THT:R_Axial_DIN0207_L6.3mm_D2.5mm_P7.62mm_Horizontal
- R17: footprint Resistors_THT:R_Axial_DIN0207_L6.3mm_D2.5mm_P10.16mm_Horizontal -> WeatherLibrary:R_Axial_DIN0207_L6.3mm_D2.5mm_P12.7mm_Horizontal
- R19: footprint Resistors_THT:R_Axial_DIN0207_L6.3mm_D2.5mm_P2.54mm_Vertical -> Resistors_THT:R_Axial_DIN0207_L6.3mm_D2.5mm_P7.62mm_Horizontal
- R3: footprint Resistors_THT:R_Axial_DIN0207_L6.3mm_D2.5mm_P7.62mm_Horizontal -> Resistors_THT:R_Axial_DIN0207_L6.3mm_D2.5mm_P5.08mm_Vertical
- R6: value 4.7k -> 1k
- Y1: footprint Crystals:Crystal_AT310_d3.0mm_l10.0mm_Vertical -> Crystals:Crystal_HC49-4H_Vertical
- moved R16 211.2 mm to (48.3, 96.5)
- moved R17 205.9 mm to (63.5, 86.4), turned to 0 degrees
- moved BT1 200.1 mm to (213.4, 66.0)
- moved Q2 200.1 mm to (256.5, 73.7)
- moved R8 200.1 mm to (256.5, 78.7)
- moved C2 200.1 mm to (238.8, 101.6)
- moved C3 200.1 mm to (238.8, 104.1)
- moved C5 200.1 mm to (243.8, 83.8)
- moved C7 200.1 mm to (243.8, 78.7)
- moved D1 200.1 mm to (251.5, 66.0)
- moved D2 200.1 mm to (251.5, 61.0)
- moved D3 200.1 mm to (238.8, 61.0)
- moved J1 200.1 mm to (269.2, 22.9)
- moved J11 200.1 mm to (231.1, 22.9)
- moved J8 200.1 mm to (238.8, 22.9)
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Connections:
- net ESP_Enable renamed /ESP_ENABLE
- net Net-(C15-Pad2) renamed /XTAL1
- net Net-(C16-Pad2) renamed /XTAL2
- net Net-(C8-Pad1) renamed /AREF
- net Net-(J3-Pad1) renamed /SCK
- net Net-(J3-Pad2) renamed /MISO
- net Net-(J3-Pad3) renamed /MOSI
- net Net-(R14-Pad1) renamed /OK_LED
- net Net-(R15-Pad1) renamed /ERROR_LED
- C1 pad 1: Anemometer -> RainBucket
- C10 pad 1: VCC -> GND
- C10 pad 2: GND -> VCC
- C11 pad 1: GND -> /AVCC
- C11 pad 2: VCC -> GND
- D3 pad 2: RefV -> GND
- D3 pad 3: GND -> RefV
- J10 pad 5: Net-(C12-Pad1) -> VCC
- J2 pad 1: GND -> VCC
- J2 pad 2: VCC -> GND
- J4 pad 5: GND -> RefV
- J4 pad 6: RefV -> DivBatV
- J4 pad 7: DivBatV -> GND
- J9 pad 1: EspResult -> EspRX
- J9 pad 2: EspRX -> EspTX
- J9 pad 3: EspTX -> GND
- J9 pad 4: EspReset -> EspSuccess
- J9 pad 5: VCC -> EspResult
- J9 pad 6: GND -> EspReset
- R3 pad 1: Anemometer -> GND
- R3 pad 2: GND -> Anemometer
- U3 pad 13: EspResult -> Net-(U3-Pad13)
- U3 pad 20: VCC -> /AVCC
- U3 pad 23: Net-(U3-Pad23) -> DivBatV
- U3 pad 24: WindVane -> RefV
- U3 pad 25: DivBatV -> Net-(U3-Pad25)
- U3 pad 26: RefV -> WindVane
- U3 pad 4: /RainBucket -> RainBucket
- U3 pad 6: EspReset -> Net-(U3-Pad6)
- U7 pad 15: Net-(U7-Pad15) -> EspReset
- U7 pad 16: EspSuccess -> EspResult
- U7 pad 17: Net-(U7-Pad17) -> EspSuccess
Routing:
- net GND: track 654.4 -> 586.1 mm, vias 28 -> 15
- net RainBucket: track 0.00 -> 62.9 mm
- net /SDA: track 95.3 -> 50.3 mm, vias 2 -> 0
- net EspReset: track 121.0 -> 77.8 mm, vias 6 -> 4
- net /SCL: track 90.6 -> 55.2 mm, vias 2 -> 0
- net EspResult: track 62.5 -> 29.5 mm
- net /OK_LED: track 27.9 -> 2.54 mm, vias 2 -> 0
- net /ERROR_LED: track 27.9 -> 2.54 mm, vias 5 -> 0
- net EspRX: track 52.3 -> 72.5 mm
- net /SRAM_CS: track 38.1 -> 18.8 mm, vias 2 -> 0
- net PanelDisable: track 15.2 -> 34.1 mm, vias 1 -> 0
- net /MISO: track 48.3 -> 29.7 mm, vias 2 -> 1
- net EspTX: track 52.3 -> 70.7 mm
- net VCC: track 437.5 -> 420.9 mm, vias 17 -> 6
- net RefVEnable: track 25.4 -> 39.2 mm
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Other:
- outline, holes or cut-outs redrawn
- net class Default: clearance 0.6 -> 0.4; trace_width 0.6 -> 0.4
- net class Power: clearance 0.6 -> 0.4; trace_width 0.6 -> 0.4
- rule trace_clearance: 0.6 -> 0.4
- board text added: "Analog Inputs"
- board text removed: "Cut Traces"

Commit message: This
Parts:
- removed Q6: FQP30N06L, TO_SOT_Packages_THT:TO-220-3_Vertical
- removed Q7: FQP27P06, TO_SOT_Packages_THT:TO-220-3_Vertical
- removed the U5 at (48.3, 119.4)
- added C6: 100nF, Capacitors_THT:C_Disc_D5.0mm_W2.5mm_P5.00mm, F.Cu at (68.6, 66.0)
- added J13: Serial, Pin_Headers:Pin_Header_Straight_1x02_Pitch2.54mm, F.Cu at (63.5, 58.4)
- added J14: Board_Power_B, Connectors_JST:JST_XH_B03B-XH-A_03x2.50mm_Straight, F.Cu at (83.8, 96.6)
- added JP2: Jumper, Pin_Headers:Pin_Header_Straight_1x02_Pitch2.54mm, F.Cu at (22.9, 55.9)
- added R25: 4.7k, Resistors_THT:R_Axial_DIN0207_L6.3mm_D2.5mm_P5.08mm_Vertical, F.Cu at (83.8, 66.0)
- C1, C4: value 10uF -> 330nF
- C10, C20, C8: footprint Capacitors_THT:C_Disc_D5.0mm_W2.5mm_P2.50mm -> Capacitors_THT:C_Disc_D5.0mm_W2.5mm_P5.00mm
- J10: footprint Connectors_JST:JST_XH_B06B-XH-A_06x2.50mm_Straight -> WeatherLibrary:JST_XH_B07B-XH-A_07x2.54mm_Straight
- J11: value Conn_01x02 -> PSU_Conn_B
- J12: footprint Connectors_JST:JST_XH_B02B-XH-A_02x2.50mm_Straight -> WeatherLibrary:JST_XH_B02B-XH-A_02x2.54mm_Straight
- J2, J7: footprint Connectors_JST:JST_XH_B04B-XH-A_04x2.50mm_Straight -> WeatherLibrary:JST_XH_B04B-XH-A_04x2.54mm_Straight
- J3: value ICSP Header -> AVR_PROG_HEADER; footprint Pin_Headers:Pin_Header_Straight_1x05_Pitch2.54mm -> Pin_Headers:Pin_Header_Straight_1x06_Pitch2.54mm
- J4: value Conn_01x05 -> Board_Power_A; footprint WeatherLibrary:JST_XH_B07B-XH-A_07x2.54mm_Straight -> WeatherLibrary:JST_XH_B04B-XH-A_04x2.54mm_Straight
- J6: footprint Connectors_JST:JST_XH_B05B-XH-A_05x2.50mm_Straight -> WeatherLibrary:JST_XH_B05B-XH-A_05x2.54mm_Straight
- J8: value Conn_01x05 -> PSU_Conn_A
- J9: footprint Connectors_JST:JST_XH_B07B-XH-A_07x2.50mm_Straight -> WeatherLibrary:JST_XH_B07B-XH-A_07x2.54mm_Straight
- L1: value 10uF -> 100uH
- R14, R15: footprint Resistors_THT:R_Axial_DIN0207_L6.3mm_D2.5mm_P15.24mm_Horizontal -> Resistors_THT:R_Axial_DIN0207_L6.3mm_D2.5mm_P7.62mm_Horizontal
- R17: footprint WeatherLibrary:R_Axial_DIN0207_L6.3mm_D2.5mm_P12.7mm_Horizontal -> Resistors_THT:R_Axial_DIN0207_L6.3mm_D2.5mm_P7.62mm_Horizontal
- R18: footprint Resistors_THT:R_Axial_DIN0207_L6.3mm_D2.5mm_P7.62mm_Horizontal -> Resistors_THT:R_Axial_DIN0207_L6.3mm_D2.5mm_P15.24mm_Horizontal
- R22: value 10K -> 4.7k
- R6: footprint Resistors_THT:R_Axial_DIN0207_L6.3mm_D2.5mm_P2.54mm_Vertical -> Resistors_THT:R_Axial_DIN0207_L6.3mm_D2.5mm_P7.62mm_Horizontal
- moved J11 131.8 mm to (170.2, 139.7), turned to 90 degrees
- moved J8 129.0 mm to (170.2, 132.1), turned to 90 degrees
- moved J1 126.5 mm to (170.2, 101.6), turned to 270 degrees
- moved R21 119.4 mm to (175.3, 121.9), turned to 270 degrees
- moved R10 117.7 mm to (177.8, 129.5), turned to 270 degrees
- moved C13 113.6 mm to (108.0, 86.3), turned to 90 degrees
- moved Q4 112.3 mm to (180.3, 121.9), turned to 90 degrees
- moved R2 111.4 mm to (185.4, 139.7), turned to 270 degrees
- moved R9 103.4 mm to (190.5, 137.2), turned to 0 degrees
- moved R5 98.0 mm to (190.5, 121.9), turned to 270 degrees
- moved C14 95.6 mm to (118.1, 86.3), turned to 90 degrees
- moved BT1 91.4 mm to (213.4, 157.5), turned to 0 degrees
- moved J5 90.3 mm to (207.0, 38.1)
- moved U4 90.3 mm to (207.0, 30.5)
- moved R22 89.3 mm to (83.8, 68.6), turned to 180 degrees
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Connections:
- C12 pad 1: Net-(C12-Pad1) -> VCC
- C13 pad 1: Net-(C12-Pad1) -> VCC
- C14 pad 1: Net-(C12-Pad1) -> VCC
- D4 pad 1: GND -> /LED_GND
- D5 pad 1: GND -> /LED_GND
- J10 pad 1: EspResult -> EspReset
- J10 pad 2: EspRX -> EspResult
- J10 pad 3: EspTX -> EspSuccess
- J10 pad 4: EspReset -> VCC
- J10 pad 5: VCC -> EspRX
- J10 pad 6: GND -> EspTX
- J3 pad 1: /SCK -> VCC
- J3 pad 2: /MISO -> /SCK
- J3 pad 3: /MOSI -> /MISO
- J3 pad 4: /Reset -> /MOSI
- J3 pad 5: GND -> /Reset
- J4 pad 1: PanelDisable -> VCC
- J4 pad 2: RefVEnable -> RefV
- J4 pad 3: BatDivEnable -> DivBatV
- J4 pad 4: VCC -> GND
- J6 pad 3: /SDA -> /SCL
- J6 pad 4: /SCL -> /SDA
- J6 pad 5: Net-(J6-Pad5) -> GND
- J7 pad 3: /SDA -> /SCL
- J7 pad 4: /SCL -> /SDA
- J9 pad 1: EspRX -> GND
- J9 pad 3: GND -> EspRX
- J9 pad 4: EspSuccess -> VCC
- J9 pad 5: EspResult -> EspSuccess
- J9 pad 6: EspReset -> EspResult
- J9 pad 7: VCC -> EspReset
- R16 pad 1: /Reset -> VCC
- R16 pad 2: VCC -> /Reset
- R20 pad 1: GND -> VCC
- R22 pad 1: Net-(C12-Pad1) -> VCC
- R22 pad 2: Net-(Q6-Pad3) -> /SDA
- U3 pad 27: /SCL -> /SDA
- U3 pad 28: /SDA -> /SCL
- U6 pad 16: Net-(U6-Pad16) -> VCC
- U6 pad 17: Net-(U6-Pad17) -> GND
- U6 pad 22: EspTX -> EspRX
- U6 pad 23: EspRX -> EspTX
- U6 pad 24: Net-(U6-Pad24) -> GND
- U6 pad 25: Net-(U6-Pad25) -> VCC
- U7 pad 1: /SDA -> /SCL
- U7 pad 18: GND -> VCC
- U7 pad 2: /SCL -> /SDA
- U7 pad 9: VCC -> GND
- U8 pad 3: /SCL -> /SDA
- U8 pad 4: /SDA -> /SCL
Routing:
- net GND: track 586.1 -> 528.4 mm, vias 15 -> 10
- net EspReset: track 77.8 -> 31.9 mm, vias 4 -> 0
- net /SRAM_CS: track 18.8 -> 56.9 mm
- net /LED_GND: track 0.00 -> 22.9 mm
- net EspResult: track 29.5 -> 7.64 mm, vias 2 -> 0
- net /Reset: track 89.2 -> 68.1 mm, vias 3 -> 0
- net Net-(C12-Pad1): track 20.3 -> 0.00 mm
- net EspRX: track 72.5 -> 55.2 mm
- net EspTX: track 70.7 -> 53.9 mm
- net WindVane: track 74.5 -> 58.0 mm, vias 1 -> 0
- net PanelDisable: track 34.1 -> 20.4 mm
- net RainBucket: track 62.9 -> 52.0 mm
- net Anemometer: track 59.8 -> 48.9 mm
- net RefVEnable: track 39.2 -> 30.5 mm
- net /SerialTX: track 0.00 -> 7.62 mm
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Other:
- board size 271.8 x 185.4 mm -> 243.8 x 134.6 mm
- net class Default: clearance 0.4 -> 0.2; trace_width 0.4 -> 0.2; via_dia 0.6 -> 0.4; via_drill 0.4 -> 0.3
- net class Power: clearance 0.4 -> 0.2; trace_width 0.4 -> 0.6
- rule trace_clearance: 0.4 -> 0.2
- rule trace_min: 0.4 -> 0.1524
- rule via_min_drill: 0.3 -> 0.254
- board text added: "7 6 5 4 3 2 1 0"
- board text added: "?!"
- board text added: "Error"
- board text added: "Esp Conn"
- board text added: "ICSP"
- board text added: "Led Enable"
- board text added: "Ok"
- board text added: "Rain"
- board text added: "Reset"
- board text added: "Serial"
- board text added: "Tower"
- board text added: "Tx Rx"
- board text added: "VCC SCK MISO MOSI RST GND"

Commit message: Schematic Updates
Parts:
- removed C12: 47uF, Capacitors_THT:CP_Radial_D5.0mm_P2.50mm
- removed C14: 470uF, Capacitors_THT:CP_Radial_D8.0mm_P2.50mm
- moved C13 19.1 mm to (127.0, 86.4)
Routing:
- net VCC: track 418.7 -> 504.8 mm
- net GND: track 528.4 -> 604.0 mm
- net EspSuccess: track 8.05 -> 73.9 mm
- net EspResult: track 7.64 -> 67.0 mm
- net EspReset: track 31.9 -> 71.0 mm
- net EspRX: track 55.2 -> 91.6 mm
- net EspTX: track 53.9 -> 89.8 mm
